Commit message: modified:   AGV_V1/rviz/AGV_V1_view.rviz 	modified:   AGV_V1/urdf/AGV_V1.urdf.xacro

File: AGV_V1/urdf/AGV_V1.urdf.xacro (robot description, xacro)
@@ -139,3 +139,19 @@
     <child link="arm_base_link"/>
   </joint>
+  <!-- Camera -->
+  <link name="camera">
+    <visual>
+      <geometry>
+        <box size="0.0125 0.05 0.0125"/> <!-- Camera dimensions -->
+      </geometry>
+      <material name="camera_material">
+        <color rgba="${camera_color}"/>
+      </material>
+    </visual>
+  </link>
+  <joint name="camera_joint" type="fixed">
+    <origin xyz="${(b_l+0.0125)/2} 0 0" rpy="0 0 0"/>
+    <parent link="upper_plate"/>
+    <child link="camera"/>
+  </joint>
 </robot>

Commit message: modified:   AGV_V1/urdf/AGV_V1.urdf.xacro

File: AGV_V1/urdf/AGV_V1.urdf.xacro (robot description, xacro)
@@ -155,3 +155,22 @@
     <child link="camera"/>
   </joint>
+  <xacro:macro name="camera_part" params="name reflect">
+    <link name="${name}">
+      <visual>
+        <geometry>
+          <cylinder length="0.005" radius="0.005"/> <!-- Camera part length and radius -->
+        </geometry>
+        <material name="base_material">
+          <color rgba="${base_color}"/>
+        </material>
+      </visual>
+    </link>
+    <joint name="${name}_joint" type="fixed">
+      <origin xyz="${0.00625} ${reflect*(0.04-0.005)/2} 0" rpy="0 ${pi/2} 0"/>
+      <parent link="camera"/>
+      <child link="${name}"/>
+    </joint>
+  </xacro:macro>
+  <xacro:camera_part name="camera_lens" reflect="1"/>
+  <xacro:camera_part name="camera_ir" reflect="-1"/>
 </robot>

Commit message: modified:   AGV_V1/urdf/AGV_V1.urdf.xacro 	new file:   AGV_V1/urdf/inertial_macros.xacro 	new file:   gazebo_worlds_sim/launch/robot.launch.py 	new file:   gazebo_worlds_sim/worlds/meshes/hexagon.dae 	new file:   gazebo_worlds_sim/worlds/meshes/wall.dae 	new file:   gazebo_worlds_sim/worlds/tb3.sdf 	modified:   robotic_manipulator/urdf/arm.urdf.xacro

File: AGV_V1/urdf/AGV_V1.urdf.xacro (robot description, xacro)
@@ -1,5 +1,7 @@
 <?xml version="1.0"?>
 <robot name="agv_with_arm" xmlns:xacro="http://ros.org/wiki/xacro">
-  <xacro:include filename="$(find robotic_manipulator)/urdf/arm.urdf.xacro"/>
+<!--
+  <xacro:include filename="$(find robotic_manipulator)/urdf/arm.urdf.xacro"/> -->
+  <xacro:include filename="$(find AGV_V1)/urdf/inertial_macros.xacro"/>
   <!-- Define colors as properties for easy modification -->
   <xacro:property name="base_color" value="0.5 0.5 0.5 1.0"/> <!-- Default gray -->
@@ -30,9 +32,15 @@
       </material>
     </visual>
+    <collision>
+      <geometry>
+        <box size="${b_l} ${b_w} ${b_h}"/> <!-- Base dimensions -->
+      </geometry>
+    </collision>
+    <xacro:inertial_solid_cuboid mass="1.0" w="${b_l}" d="${b_w}" h="${b_h}"/>
   </link>
   <joint name="base_footprint_joint" type="fixed">
     <parent link="base_footprint"/>
     <child link="base_link"/>
-    <origin xyz="0 0 0.1"/> <!-- Base height -->
+    <origin xyz="0 0 ${b_h}"/> <!-- Base height -->
   </joint>
   <!-- Wheel -->
@@ -47,4 +55,10 @@
         </material>
       </visual>
+      <collision>
+        <geometry>
+          <cylinder length="${w_l}" radius="${w_r}"/> <!-- Wheel height and radius -->
+        </geometry>
+      </collision>
+      <xacro:inertial_solid_cylinder mass="1.0" r="${w_r}" h="${w_l}"/>
     </link>
     <joint name="${name}_wheel_joint" type="continuous">
@@ -90,4 +104,10 @@
         </material>
       </visual>
+      <collision>
+        <geometry>
+          <box size="${w_r/2} ${w_r/2} ${w_r}"/> <!-- Pillar height and radius -->
+        </geometry>
+      </collision>
+      <xacro:inertial_solid_cuboid mass="1.0" w="${w_r/2}" d="${w_r/2}" h="${w_r}"/>
     </link>
     <joint name="${name}_pillar_joint" type="fixed">
@@ -111,4 +131,10 @@
       </material>
     </visual>
+    <collision>
+      <geometry>
+        <cylinder length="${lidar_l}" radius="${lidar_r}"/> <!-- Lidar length and radius -->
+      </geometry>
+    </collision>
+    <xacro:inertial_solid_cylinder mass="1.0" r="${lidar_r}" h="${lidar_l}"/>
   </link>
   <joint name="lidar_joint" type="fixed">
@@ -127,4 +153,10 @@
       </material>
     </visual>
+    <collision>
+      <geometry>
+        <box size="${b_l} ${b_w} ${upper_plate_h}"/> <!-- Upper plate dimensions -->
+      </geometry>
+    </collision>
+    <xacro:inertial_solid_cuboid mass="1.0" w="${b_l}" d="${b_w}" h="${upper_plate_h}"/>
   </link>
   <joint name="upper_plate_joint" type="fixed">
@@ -133,10 +165,10 @@
     <child link="upper_plate"/>
   </joint>
-  <!-- Arm -->
+  <!-- Arm
   <joint name="arm_base_joint" type="fixed">
     <origin xyz="${(b_l/2)-cylinder_radius} 0 0" rpy="0 0 0"/>
     <parent link="upper_plate"/>
     <child link="arm_base_link"/>
-  </joint>
+  </joint>-->
   <!-- Camera -->
   <link name="camera">
@@ -149,4 +181,10 @@
       </material>
     </visual>
+    <collision>
+      <geometry>
+        <box size="0.0125 0.05 0.0125"/> <!-- Camera dimensions -->
+      </geometry>
+    </collision>
+    <xacro:inertial_solid_cuboid mass="1.0" w="0.0125" d="0.05" h="0.0125"/>
   </link>
   <joint name="camera_joint" type="fixed">
@@ -165,4 +203,10 @@
         </material>
       </visual>
+      <collision>
+        <geometry>
+          <cylinder length="0.005" radius="0.005"/> <!-- Camera part length and radius -->
+        </geometry>
+      </collision>
+      <xacro:inertial_solid_cylinder mass="1.0" r="0.005" h="0.005"/>
     </link>
     <joint name="${name}_joint" type="fixed">

File: robotic_manipulator/urdf/arm.urdf.xacro (robot description, xacro)
@@ -1,4 +1,5 @@
 <?xml version="1.0"?>
 <robot xmlns:xacro="http://www.ros.org/wiki/xacro" name="five_dof_manipulator_with_gripper">
+  <xacro:include filename="$(find AGV_V1)/urdf/inertial_macros.xacro"/>
   <!-- Define properties -->
   <xacro:property name="cylinder_radius" value="0.05"/>
@@ -19,4 +20,11 @@
         </material>
       </visual>
+      <collision>
+        <origin xyz="0 0 ${length/2}" rpy="0 0 0"/>
+        <geometry>
+          <cylinder radius="${radius}" length="${length}"/>
+        </geometry>
+      </collision>
+      <xacro:inertial_solid_cylinder mass="0.01" r="${radius}" h="${length}"/>
     </link>
   </xacro:macro>
@@ -50,4 +58,11 @@
         </material>
       </visual>
+      <collision>
+        <origin xyz="0 0.015 0" rpy="0 0 0"/>
+        <geometry>
+          <box size="0.01 0.01 0.05"/>
+        </geometry>
+      </collision>
+      <xacro:inertial_solid_cuboid mass="0.005" w="0.01" d="0.01" h="0.05"/>
     </link>
   </xacro:macro>
@@ -78,4 +93,11 @@
       </material>
     </visual>
+    <collision>
+      <origin xyz="0 0 0" rpy="0 0 0"/>
+      <geometry>
+        <box size="0.05 0.025 0.05"/>
+      </geometry>
+    </collision>
+    <xacro:inertial_solid_cuboid mass="0.01" w="0.05" d="0.025" h="0.05"/>
   </link>
   <!-- Gripper Fingers -->

Commit message: modified:   AGV_V1/urdf/AGV_V1.urdf.xacro 	modified:   AGV_V1/urdf/AGV_V1_gz.urdf.xacro 	new file:   d435i_depth

File: AGV_V1/urdf/AGV_V1.urdf.xacro (robot description, xacro)
@@ -4,4 +4,5 @@
   <xacro:include filename="$(find robotic_manipulator)/urdf/arm.urdf.xacro"/> -->
   <xacro:include filename="$(find AGV_V1)/urdf/inertial_macros.xacro"/>
+  <xacro:include filename="$(find d435i_depth)/urdf/d435i_gz.urdf.xacro"/>
   <!-- Define colors as properties for easy modification -->
   <xacro:property name="base_color" value="0.5 0.5 0.5 1.0"/> <!-- Default gray -->
@@ -171,9 +172,9 @@
     <child link="arm_base_link"/>
   </joint>-->
-  <!-- Camera -->
+  <!-- Camera
   <link name="camera">
     <visual>
       <geometry>
-        <box size="0.0125 0.05 0.0125"/> <!-- Camera dimensions -->
+        <box size="0.0125 0.05 0.0125"/> Camera dimensions
       </geometry>
       <material name="camera_material">
@@ -183,5 +184,5 @@
     <collision>
       <geometry>
-        <box size="0.0125 0.05 0.0125"/> <!-- Camera dimensions -->
+        <box size="0.0125 0.05 0.0125"/> amera dimensions
       </geometry>
     </collision>
@@ -197,5 +198,5 @@
       <visual>
         <geometry>
-          <cylinder length="0.005" radius="0.005"/> <!-- Camera part length and radius -->
+          <cylinder length="0.005" radius="0.005"/> Camera part length and radius
         </geometry>
         <material name="base_material">
@@ -205,5 +206,5 @@
       <collision>
         <geometry>
-          <cylinder length="0.005" radius="0.005"/> <!-- Camera part length and radius -->
+          <cylinder length="0.005" radius="0.005"/> Camera part length and radius
         </geometry>
       </collision>
@@ -217,4 +218,9 @@
   </xacro:macro>
   <xacro:camera_part name="camera_lens" reflect="1"/>
-  <xacro:camera_part name="camera_ir" reflect="-1"/>
+  <xacro:camera_part name="camera_ir" reflect="-1"/> -->
+  <joint name="d_cam_joint" type="fixed">
+    <origin xyz="${(b_l+0.0125)/2-0.01} 0 0.0055" rpy="0 0 0"/>
+    <parent link="upper_plate"/>
+    <child link="base_screw"/>
+  </joint>
 </robot>

File: AGV_V1/urdf/AGV_V1_gz.urdf.xacro (robot description, xacro)
@@ -3,26 +3,31 @@
     <xacro:include filename="$(find AGV_V1)/urdf/AGV_V1.urdf.xacro"/>
     <!--Gazebo Plugins-->
-    <gazebo>
-        <plugin name="skid_steer_drive_controller" filename="libgazebo_ros_skid_steer_drive.so">
-            <updateRate>100.0</updateRate>
-            <robotNamespace>/</robotNamespace>
-            <leftFrontJoint>front_left</leftFrontJoint>
-            <rightFrontJoint>front_right</rightFrontJoint>
-            <leftRearJoint>back_left</leftRearJoint>
-            <rightRearJoint>back_right</rightRearJoint>
-            <wheelSeparation>0.275</wheelSeparation>
-            <wheelDiameter>0.1</wheelDiameter>
-            <robotBaseFrame>base_link</robotBaseFrame>
-            <torque>20</torque>
-            <topicName>cmd_vel</topicName>
-            <broadcastTF>false</broadcastTF>
-            <publish_odom>true</publish_odom>
-            <publish_odom_tf>true</publish_odom_tf>
-            <publish_wheel_tf>true</publish_wheel_tf>
-            <odometry_frame>/odom</odometry_frame>
-            <robot_base_frame>base_link</robot_base_frame>
-        </plugin>
-    </gazebo>
-    <gazebo>
+  <gazebo>
+    <plugin name="ros2_control" filename="libros2_control_gazebo.so">
+      <robotNamespace>AGV</robotNamespace>
+    </plugin>
+  </gazebo>
+  <gazebo>
+      <plugin filename="ignition-gazebo-diff-drive-system" name="ignition::gazebo::systems::DiffDrive">
+        <!-- Wheel Joints -->
+        <left_joint>front_left</left_joint>
+        <right_joint>front_right</right_joint>
+        <left_joint>back_left</left_joint>
+        <right_joint>back_right</right_joint>
+        <!-- Kinematics -->
+        <wheel_separation>0.275</wheel_separation>
+        <wheel_radius>0.05</wheel_radius>
+        <odom_publish_frequency>200</odom_publish_frequency>
+        <!-- TF Frames -->
+        <frame_id>/odom</frame_id>
+        <child_frame_id>/base_link</child_frame_id>
+        <!-- topics -->
+        <topic>/AGV/cmd_vel</topic>
+        <odom_topic>/AGV/odometry</odom_topic>
+        <tf_topic>/AGV/tf</tf_topic>
+        <tf_topic></tf_topic>
+      </plugin>
+  </gazebo>
+  <gazebo>
       <plugin filename="ignition-gazebo-joint-state-publisher-system" name="ignition::gazebo::systems::JointStatePublisher">
         <update_rate>100</update_rate>
@@ -130,44 +135,3 @@
     </sensor>
   </gazebo>
-  <gazebo reference="camera">
-  <sensor name="camera_lens" type="depth">
-    <update_rate>20</update_rate>
-    <camera>
-      <horizontal_fov>1.047198</horizontal_fov>
-      <image>
-        <width>640</width>
-        <height>480</height>
-        <format>R8G8B8</format>
-      </image>
-      <clip>
-        <near>0.05</near>
-        <far>3</far>
-      </clip>
-    </camera>
-    <plugin name="camera_ir" filename="libgazebo_ros_openni_kinect.so">
-      <baseline>0.2</baseline>
-      <alwaysOn>true</alwaysOn>
-      <updateRate>1.0</updateRate>
-      <cameraName>AGV_camera_ir</cameraName>
-      <imageTopicName>/AGV_camera/color/image_raw</imageTopicName>
-      <cameraInfoTopicName>/AGV_camera/color/camera_info</cameraInfoTopicName>
-      <depthImageTopicName>/AGV_camera/depth/image_raw</depthImageTopicName>
-      <depthImageInfoTopicName>/AGV_camera/depth/camera_info</depthImageInfoTopicName>
-      <pointCloudTopicName>/AGV_camera/depth/points</pointCloudTopicName>
-      <frameName>camera</frameName>
-      <pointCloudCutoff>0.5</pointCloudCutoff>
-      <pointCloudCutoffMax>3.0</pointCloudCutoffMax>
-      <distortionK1>0.00000001</distortionK1>
-      <distortionK2>0.00000001</distortionK2>
-      <distortionK3>0.00000001</distortionK3>
-      <distortionT1>0.00000001</distortionT1>
-      <distortionT2>0.00000001</distortionT2>
-      <CxPrime>0</CxPrime>
-      <Cx>0</Cx>
-      <Cy>0</Cy>
-      <focalLength>0</focalLength>
-      <hackBaseline>0</hackBaseline>
-    </plugin>
-  </sensor>
-  </gazebo>
 </robot>
