Commit message: modified:   AGV_V1/launch/agv_v1.launch.py 	modified:   AGV_V1/rviz/AGV_V1_view.rviz 	renamed:    AGV_V1/urdf/AGV_V1_gz.urdf.xacro -> AGV_V1/urdf/AGV_V1.gazebo.xacro 	modified:   AGV_V1/urdf/AGV_V1.urdf.xacro 	new file:   AGV_V2/CMakeLists.txt 	new file:   AGV_V2/launch/agv_v2.launch.py 	new file:   AGV_V2/package.xml 	modified:   d435i_depth 	modified:   gazebo_worlds_sim/launch/robot.launch.py
 Changes not staged for commit:
	modified:   d435i_depth (modified content, untracked content)

File: AGV_V1/urdf/AGV_V1.gazebo.xacro (robot description, xacro)
@@ -1,44 +1,40 @@
 <?xml version="1.0"?>
-<robot name="agv" xmlns:xacro="http://ros.org/wiki/xacro">
-    <xacro:include filename="$(find AGV_V1)/urdf/AGV_V1.urdf.xacro"/>
-    <!--Gazebo Plugins-->
+<robot xmlns:xacro="http://ros.org/wiki/xacro">
+  <!-- ros_control plugin -->
   <gazebo>
     <plugin name="ros2_control" filename="libros2_control_gazebo.so">
-      <robotNamespace>AGV</robotNamespace>
+      <robotNamespace>$(arg robot_ns)</robotNamespace>
     </plugin>
   </gazebo>
+  <!-- Differential Drive - https://gazebosim.org/api/gazebo/4.5/classignition_1_1gazebo_1_1systems_1_1DiffDrive.html -->
   <gazebo>
-      <plugin filename="ignition-gazebo-diff-drive-system" name="ignition::gazebo::systems::DiffDrive">
-        <!-- Wheel Joints -->
-        <left_joint>front_left</left_joint>
-        <right_joint>front_right</right_joint>
-        <left_joint>back_left</left_joint>
-        <right_joint>back_right</right_joint>
-        <!-- Kinematics -->
-        <wheel_separation>0.275</wheel_separation>
-        <wheel_radius>0.05</wheel_radius>
-        <odom_publish_frequency>200</odom_publish_frequency>
-        <!-- TF Frames -->
-        <frame_id>/odom</frame_id>
-        <child_frame_id>/base_link</child_frame_id>
-        <!-- topics -->
-        <topic>/AGV/cmd_vel</topic>
-        <odom_topic>/AGV/odometry</odom_topic>
-        <tf_topic>/AGV/tf</tf_topic>
-        <tf_topic></tf_topic>
-      </plugin>
+    <plugin filename="ignition-gazebo-diff-drive-system" name="ignition::gazebo::systems::DiffDrive">
+      <!-- Wheel Joints -->
+      <left_joint>left_wheel_joint</left_joint>
+      <right_joint>right_wheel_joint</right_joint>
+      <!-- Kinematics -->
+      <wheel_separation>0.275</wheel_separation>
+      <wheel_radius>0.05</wheel_radius>
+      <odom_publish_frequency>200</odom_publish_frequency>
+      <!-- TF Frames -->
+      <frame_id>/odom</frame_id>
+      <child_frame_id>/base_link</child_frame_id>
+      <!-- topics -->
+      <topic>/model/leo/cmd_vel</topic>
+      <odom_topic>/model/leo/odometry</odom_topic>
+      <tf_topic>/model/leo/tf</tf_topic>
+      <tf_topic></tf_topic>
+    </plugin>
   </gazebo>
   <gazebo>
       <plugin filename="ignition-gazebo-joint-state-publisher-system" name="ignition::gazebo::systems::JointStatePublisher">
         <update_rate>100</update_rate>
-        <joint_name>front_left</joint_name>
-        <joint_name>front_right</joint_name>
-        <joint_name>back_left</joint_name>
-        <joint_name>back_right</joint_name>
+        <joint_name>left_wheel_joint</joint_name>
+        <joint_name>right_wheel_joint</joint_name>
       </plugin>
   </gazebo>
   <gazebo reference="base_link">
     <sensor name="imu_sensor" type="imu">
-      <topic>/AGV/imu</topic>
+      <topic>/model/leo/imu</topic>
       <frame_id>base_link</frame_id>
       <ignition_frame_id>base_link</ignition_frame_id>
@@ -105,9 +101,10 @@
     </sensor>
   </gazebo>
-  <gazebo reference="lidar">
+  <!--lidar-->
+  <gazebo reference="lidar_link">
     <sensor type="gpu_lidar" name="generic_lidar_sensor">
-      <topic>/AGV/scan</topic>
-      <frame_id>lidar</frame_id>
-      <ignition_frame_id>lidar</ignition_frame_id>
+      <topic>/model/leo/scan</topic>
+      <frame_id>lidar_link</frame_id>
+      <ignition_frame_id>lidar_link</ignition_frame_id>
       <update_rate>20.0</update_rate>
       <ray>

File: AGV_V1/urdf/AGV_V1.urdf.xacro (robot description, xacro)
@@ -1,8 +1,9 @@
 <?xml version="1.0"?>
-<robot name="agv_with_arm" xmlns:xacro="http://ros.org/wiki/xacro">
+<robot name="agv" xmlns:xacro="http://ros.org/wiki/xacro">
 <!--
   <xacro:include filename="$(find robotic_manipulator)/urdf/arm.urdf.xacro"/> -->
+  <xacro:arg name="robot_ns" default="agv"/>
   <xacro:include filename="$(find AGV_V1)/urdf/inertial_macros.xacro"/>
-  <xacro:include filename="$(find d435i_depth)/urdf/d435i_gz.urdf.xacro"/>
+  <xacro:include filename="$(find d435i_depth)/urdf/test_d435i.urdf.xacro"/>
   <!-- Define colors as properties for easy modification -->
   <xacro:property name="base_color" value="0.5 0.5 0.5 1.0"/> <!-- Default gray -->
@@ -23,5 +24,4 @@
   <xacro:property name="upper_plate_h" value="0.0125"/> <!-- Upper plate height -->
   <!-- Base Link (Chassis) -->
-  <link name="base_footprint"/>
   <link name="base_link">
     <visual>
@@ -40,9 +40,4 @@
     <xacro:inertial_solid_cuboid mass="1.0" w="${b_l}" d="${b_w}" h="${b_h}"/>
   </link>
-  <joint name="base_footprint_joint" type="fixed">
-    <parent link="base_footprint"/>
-    <child link="base_link"/>
-    <origin xyz="0 0 ${b_h}"/> <!-- Base height -->
-  </joint>
   <!-- Wheel -->
   <xacro:macro name="wheel" params="name x_reflect y_reflect">
@@ -64,5 +59,5 @@
     </link>
     <joint name="${name}_wheel_joint" type="continuous">
-      <origin xyz="${x_reflect*b_l/2} ${y_reflect*(b_w+w_l)/2} ${-b_h/2}" rpy="${-pi/2} 0 0"/>
+      <origin xyz="${0*x_reflect*b_l/2} ${y_reflect*(b_w+w_l)/2} ${-b_h/2}" rpy="${-pi/2} 0 0"/>
       <parent link="base_link"/>
       <child link="${name}_wheel"/>
@@ -70,9 +65,7 @@
     </joint>
   </xacro:macro>
-  <xacro:wheel name="front_left" x_reflect="1" y_reflect="1"/>
-  <xacro:wheel name="front_right" x_reflect="1" y_reflect="-1"/>
-  <xacro:wheel name="back_left" x_reflect="-1" y_reflect="1"/>
-  <xacro:wheel name="back_right" x_reflect="-1" y_reflect="-1"/>
-  <!-- Caster Wheel
+  <xacro:wheel name="left" x_reflect="1" y_reflect="1"/>
+  <xacro:wheel name="right" x_reflect="1" y_reflect="-1"/>
+  <!-- Caster Wheel -->
   <xacro:macro name="caster_wheel" params="name reflect">
     <link name="${name}_caster_wheel">
@@ -85,7 +78,13 @@
         </material>
       </visual>
+      <collision>
+        <geometry>
+          <sphere radius="0.05"/>
+        </geometry>
+      </collision>
+      <xacro:inertial_solid_sphere mass="1.0" r="0.05"/>
     </link>
     <joint name="${name}_caster_wheel_joint" type="fixed">
-      <origin xyz="${reflect*0.25} 0 -0.1" rpy="0 0 0"/>
+      <origin xyz="${reflect*(b_l/2-w_r)} 0 ${-b_h/2}" rpy="0 0 0"/>
       <parent link="base_link"/>
       <child link="${name}_caster_wheel"/>
@@ -93,5 +92,5 @@
   </xacro:macro>
   <xacro:caster_wheel name="front" reflect="1"/>
-  <xacro:caster_wheel name="back" reflect="-1"/> -->
+  <xacro:caster_wheel name="back" reflect="-1"/>
   <!-- Pillar-->
   <xacro:macro name="pillar" params="name x_reflect y_reflect">
@@ -123,5 +122,5 @@
   <xacro:pillar name="back_right" x_reflect="-1" y_reflect="-1"/>
   <!-- Lidar -->
-  <link name="lidar">
+  <link name="lidar_link">
     <visual>
       <geometry>
@@ -142,5 +141,5 @@
     <origin xyz="0 0 ${(b_h+lidar_l)/2}" rpy="0 0 0"/>
     <parent link="base_link"/>
-    <child link="lidar"/>
+    <child link="lidar_link"/>
   </joint>
   <!--Upper Plate-->
@@ -224,3 +223,10 @@
     <child link="base_screw"/>
   </joint>
+  <link name="base_footprint"/>
+  <joint name="base_footprint_joint" type="fixed">
+    <origin xyz="0 0 ${b_h}"/> <!-- Base height -->
+    <parent link="base_footprint"/>
+    <child link="base_link"/>
+  </joint>
+  <xacro:include filename="$(find AGV_V1)/urdf/AGV_V1.gazebo.xacro"/>
 </robot>
