Commit message: new file:   .vscode/c_cpp_properties.json 	deleted:    AGV_V1/urdf/AGV_V1.gazebo.xacro 	deleted:    AGV_V2/launch/agv_v2.launch.py 	renamed:    AGV_V1/CMakeLists.txt -> agv_v1/CMakeLists.txt 	new file:   agv_v1/config/agv_ros2_control.yaml 	renamed:    AGV_V1/launch/agv_v1.launch.py -> agv_v1/launch/agv_v1.launch.py 	renamed:    AGV_V1/package.xml -> agv_v1/package.xml 	renamed:    AGV_V1/rviz/AGV_V1_view.rviz -> agv_v1/rviz/agv_v1_view.rviz 	new file:   agv_v1/urdf/agv_v1.gazebo.xacro 	renamed:    AGV_V1/urdf/AGV_V1.urdf.xacro -> agv_v1/urdf/agv_v1.urdf.xacro 	renamed:    AGV_V1/urdf/inertial_macros.xacro -> agv_v1/urdf/inertial_macros.xacro 	new file:   agv_v2/CMakeLists.txt 	new file:   agv_v2/config/twist_mux_params.yaml 	new file:   agv_v2/include/PointCloudPublisher.hpp 	new file:   agv_v2/launch/agv_v2.launch.py 	renamed:    AGV_V2/package.xml -> agv_v2/package.xml 	new file:   agv_v2/src/PointCloudPublisher.cpp 	new file:   agv_v2/src/arm_trajectory_publisher.py 	renamed:    AGV_V2/CMakeLists.txt -> agv_v3/CMakeLists.txt 	new file:   agv_v3/package.xml 	deleted:    d435i_depth 	new file:   realsense_cam 	modified:   robotic_manipulator/CMakeLists.txt 	new file:   robotic_manipulator/config/arm_controllers.yaml 	modified:   robotic_manipulator/launch/arm.launch.py 	new file:   robotic_manipulator/urdf/arm.gazebo.xacro 	modified:   robotic_manipulator/urdf/arm.urdf.xacro

File: agv_v1/urdf/agv_v1.urdf.xacro (robot description, xacro)
@@ -4,6 +4,7 @@
   <xacro:include filename="$(find robotic_manipulator)/urdf/arm.urdf.xacro"/> -->
   <xacro:arg name="robot_ns" default="agv"/>
-  <xacro:include filename="$(find AGV_V1)/urdf/inertial_macros.xacro"/>
-  <xacro:include filename="$(find d435i_depth)/urdf/test_d435i.urdf.xacro"/>
+  <xacro:include filename="$(find agv_v1)/urdf/inertial_macros.xacro"/>
+  <!-- <xacro:include filename="$(find realsense_cam)/urdf/test_d435i.urdf.xacro"/> -->
+  <xacro:include filename="$(find robotic_manipulator)/urdf/arm.urdf.xacro"/>
   <!-- Define colors as properties for easy modification -->
   <xacro:property name="base_color" value="0.5 0.5 0.5 1.0"/> <!-- Default gray -->
@@ -18,4 +19,6 @@
   <xacro:property name="w_r" value="0.05"/> <!-- Wheel radius -->
   <xacro:property name="w_l" value="0.025"/> <!-- Wheel length -->
+  <xacro:property name="s_r" value="0.01"/>
+  <xacro:property name="s_l" value="0.075"/>
   <xacro:property name="lidar_r" value="0.025"/> <!-- Lidar radius -->
   <xacro:property name="lidar_l" value="0.025"/> <!-- Lidar length -->
@@ -40,4 +43,56 @@
     <xacro:inertial_solid_cuboid mass="1.0" w="${b_l}" d="${b_w}" h="${b_h}"/>
   </link>
+  <!--Steering link-->
+  <xacro:macro name="steering_link1" params="name x_reflect y_reflect">
+    <link name="${name}_steering_link">
+      <visual>
+        <geometry>
+          <cylinder length="${s_l}" radius="${s_r}"/>
+        </geometry>
+        <material name="base_material">
+          <color rgba="${base_color}"/>
+        </material>
+      </visual>
+      <collision>
+        <geometry>
+          <cylinder length="${s_l}" radius="${s_r}"/>
+        </geometry>
+      </collision>
+      <xacro:inertial_solid_cylinder mass="1.0" r="${s_r}" h="${s_l}"/>
+    </link>
+    <joint name="${name}_steering_joint" type="continuous">
+      <origin xyz="${x_reflect*(b_l-(2*s_r))/2} ${y_reflect*(b_w)/2} ${(-b_h/2) + s_r}" rpy="${-pi/2} 0 0"/>
+      <parent link="base_link"/>
+      <child link="${name}_steering_link"/>
+      <axis xyz="0 0 1"/>
+    </joint>
+  </xacro:macro>
+  <xacro:steering_link1 name="front_left" x_reflect="1" y_reflect="1"/>
+  <xacro:steering_link1 name="front_right" x_reflect="1" y_reflect="-1"/>
+  <xacro:macro name="steering_link2" params="name x_reflect y_reflect">
+    <link name="${name}_steering_link">
+      <visual>
+        <geometry>
+          <cylinder length="${s_l}" radius="${s_r}"/>
+        </geometry>
+        <material name="base_material">
+          <color rgba="${base_color}"/>
+        </material>
+      </visual>
+      <collision>
+        <geometry>
+          <cylinder length="${s_l}" radius="${s_r}"/>
+        </geometry>
+      </collision>
+      <xacro:inertial_solid_cylinder mass="1.0" r="${s_r}" h="${s_l}"/>
+    </link>
+    <joint name="${name}_steering_joint" type="fixed">
+      <origin xyz="${x_reflect*(b_l-(2*s_r))/2} ${y_reflect*(b_w)/2} ${(-b_h/2) + s_r}" rpy="${-pi/2} 0 0"/>
+      <parent link="base_link"/>
+      <child link="${name}_steering_link"/>
+    </joint>
+  </xacro:macro>
+  <xacro:steering_link2 name="back_left" x_reflect="-1" y_reflect="1"/>
+  <xacro:steering_link2 name="back_right" x_reflect="-1" y_reflect="-1"/>
   <!-- Wheel -->
   <xacro:macro name="wheel" params="name x_reflect y_reflect">
@@ -59,13 +114,15 @@
     </link>
     <joint name="${name}_wheel_joint" type="continuous">
-      <origin xyz="${0*x_reflect*b_l/2} ${y_reflect*(b_w+w_l)/2} ${-b_h/2}" rpy="${-pi/2} 0 0"/>
-      <parent link="base_link"/>
+      <origin xyz="0 0 ${y_reflect*(s_l/2)}" rpy="0 0 0"/>
+      <parent link="${name}_steering_link"/>
       <child link="${name}_wheel"/>
       <axis xyz="0 0 1"/>
     </joint>
   </xacro:macro>
-  <xacro:wheel name="left" x_reflect="1" y_reflect="1"/>
-  <xacro:wheel name="right" x_reflect="1" y_reflect="-1"/>
-  <!-- Caster Wheel -->
+  <xacro:wheel name="front_left" x_reflect="1" y_reflect="1"/>
+  <xacro:wheel name="front_right" x_reflect="1" y_reflect="-1"/>
+  <xacro:wheel name="back_left" x_reflect="-1" y_reflect="1"/>
+  <xacro:wheel name="back_right" x_reflect="-1" y_reflect="-1"/>
+  <!-- Caster Wheel
   <xacro:macro name="caster_wheel" params="name reflect">
     <link name="${name}_caster_wheel">
@@ -93,4 +150,5 @@
   <xacro:caster_wheel name="front" reflect="1"/>
   <xacro:caster_wheel name="back" reflect="-1"/>
+  -->
   <!-- Pillar-->
   <xacro:macro name="pillar" params="name x_reflect y_reflect">
@@ -218,4 +276,5 @@
   <xacro:camera_part name="camera_lens" reflect="1"/>
   <xacro:camera_part name="camera_ir" reflect="-1"/> -->
+  <!--
   <joint name="d_cam_joint" type="fixed">
     <origin xyz="${(b_l+0.0125)/2-0.01} 0 0.0055" rpy="0 0 0"/>
@@ -223,10 +282,10 @@
     <child link="base_screw"/>
   </joint>
-  <link name="base_footprint"/>
-  <joint name="base_footprint_joint" type="fixed">
-    <origin xyz="0 0 ${b_h}"/> <!-- Base height -->
-    <parent link="base_footprint"/>
-    <child link="base_link"/>
-  </joint>
-  <xacro:include filename="$(find AGV_V1)/urdf/AGV_V1.gazebo.xacro"/>
+  -->
+  <joint name="arm_joint" type="fixed">
+    <origin xyz="${(b_l)/2-0.05} 0 0.0055" rpy="0 0 0"/>
+    <parent link="upper_plate"/>
+    <child link="arm_base_link"/>
+  </joint>
+  <xacro:include filename="$(find agv_v1)/urdf/agv_v1.gazebo.xacro"/>
 </robot>

File: robotic_manipulator/urdf/arm.urdf.xacro (robot description, xacro)
@@ -1,5 +1,6 @@
 <?xml version="1.0"?>
 <robot xmlns:xacro="http://www.ros.org/wiki/xacro" name="five_dof_manipulator_with_gripper">
-  <xacro:include filename="$(find AGV_V1)/urdf/inertial_macros.xacro"/>
+  <xacro:include filename="$(find agv_v1)/urdf/inertial_macros.xacro"/>
+  <xacro:include filename="$(find realsense_cam)/urdf/test_d435i.urdf.xacro"/>
   <!-- Define properties -->
   <xacro:property name="cylinder_radius" value="0.05"/>
@@ -104,3 +105,8 @@
   <xacro:gripper_finger finger_name="finger_1" offset="0.02 0 0" direction="0.05"/>
   <xacro:gripper_finger finger_name="finger_2" offset="-0.02 0 0" direction="-0.05"/>
+  <joint name="d_cam_joint" type="fixed">
+    <origin xyz="0 0 -0.025" rpy="${pi} 0 ${pi/2}"/>
+    <parent link="gripper_base"/>
+    <child link="base_screw"/>
+  </joint>
 </robot>
